Commit message: checkpoint: benchmarking complete, before Gazebo attach fix attempt

File: franka_description/robots/common/franka_arm.srdf.xacro (robot description, xacro)
@@ -4,5 +4,5 @@
         <xacro:property name="prefix" value="${'' if no_prefix else arm_prefix + robot_type + '_'}" />
         <xacro:include filename="$(find franka_description)/robots/common/group_definition.xacro"/>
-        <xacro:property name="tip_link" value="${prefix + 'hand_tcp' if hand and ee_id == 'franka_hand' else prefix + 'link8'}"/>
+        <xacro:property name="tip_link" value="${prefix + 'hand_tcp' if hand and ee_id == 'franka_hand' else prefix + ee_id + '_tcp' if hand else prefix + 'link8'}"/>
         <xacro:group_definition prefix="${prefix}" group_name="${prefix}arm" tip_link="${tip_link}"/>
         <virtual_joint name="virtual_joint" type="fixed" parent_frame="world" child_link="base"/>
@@ -35,4 +35,9 @@
                 <xacro:franka_hand_srdf prefix="${prefix}"/>
             </xacro:if>
+            <xacro:unless value="${ee_id == 'franka_hand'}">
+                <disable_collisions link1="${prefix}link7" link2="${prefix}${ee_id}" reason="Adjacent"/>
+                <disable_collisions link1="${prefix}link8" link2="${prefix}${ee_id}" reason="Adjacent"/>
+                <disable_collisions link1="${prefix}link6" link2="${prefix}${ee_id}" reason="Never"/>
+            </xacro:unless>
         </xacro:if>
     </xacro:macro>
