Commit message: fix(gazebo): decouple box and pump collision and add detachable joint plugin

File: franka_description/end_effectors/cobot_pump/cobot_pump.urdf.xacro (robot description, xacro)
@@ -17,3 +17,11 @@
                           with_sc="$(arg with_sc)">
    </xacro:ee_with_one_link>
+  <xacro:property name="ee_prefix" value="${robot_type}_" />
+  <gazebo reference="${ee_prefix}${ee_id}_collision">
+    <surface>
+      <contact>
+        <collide_bitmask>0x02</collide_bitmask>
+      </contact>
+    </surface>
+  </gazebo>
 </robot>

Commit message: feat(gazebo): dynamic obstacle spawning, CHOMP planner support, and Gazebo-physics benchmarks
Adds fast_detach_node and a ros_gz_bridge for box attach/detach, spawns the
Part 3 obstacle live in Gazebo instead of only in the MoveIt scene, wires
planner_id (RRTConnect/CHOMP) through pick_place.launch.py, and adds
obstacle world variants plus scripts/results for Gazebo-physics benchmarking.

File: franka_description/end_effectors/cobot_pump/cobot_pump.urdf.xacro (robot description, xacro)
@@ -17,11 +17,12 @@
                           with_sc="$(arg with_sc)">
    </xacro:ee_with_one_link>
-  <xacro:property name="ee_prefix" value="${robot_type}_" />
-  <gazebo reference="${ee_prefix}${ee_id}_collision">
-    <surface>
-      <contact>
-        <collide_bitmask>0x02</collide_bitmask>
-      </contact>
-    </surface>
+  <gazebo reference="fr3_cobot_pump">
+    <collision name="fr3_cobot_pump_collision">
+      <surface>
+        <contact>
+          <collide_bitmask>0x02</collide_bitmask>
+        </contact>
+      </surface>
+    </collision>
   </gazebo>
 </robot>

File: franka_description/robots/fr3/fr3.urdf.xacro (robot description, xacro)
@@ -64,3 +64,12 @@
     connected_to="base">
   </xacro:franka_robot>
+  <gazebo reference="fr3_cobot_pump">
+    <collision name="fr3_cobot_pump_collision">
+      <surface>
+        <contact>
+          <collide_bitmask>0x02</collide_bitmask>
+        </contact>
+      </surface>
+    </collision>
+  </gazebo>
 </robot>
